File: 3) Hardware/PCB Design/1) Prototype Circuit Design (V3)/ThrusterV3/ThrusterV3.kicad_sch (KiCad schematic)
At the start: 77 parts, among them J1 Conn_01x06_Pin, J2 Conn_01x02_Pin, J3 Conn_01x02_Pin, J4 Conn_01x02_Pin, J5 Conn_01x02_Pin, J6 Conn_01x02_Pin, J7 Conn_01x04_Pin, J8 USB_C_Receptacle, J9 Conn_01x04_Pin, Q1 AO3400A, Q2 AO3400A, Q3 AO3400A, Q4 AO3400A, Q5 AO3400A, Q6 IPD70P04P4L08ATMA2, SW1 SW_Push, U1 INA126U, U2 STM32G491CCTx, U3 AP63205WU, U4 AMS1117-3.3, U5 ADS131M04IPWR, U6 MCP6024-E_SL, Y1 8MHz

Commit message: Finished Routing Thruster V3 PCB
Parts:
- removed J8: USB_C_Receptacle, Connector_USB:USB_C_Receptacle_Molex_105450-0101, symbol Connector:USB_C_Receptacle
- removed R1: 10k, Resistor_SMD:R_0603_1608Metric, symbol Device:R
- added C20, C24, C30, C31, C32, C33: 100n, Capacitor_SMD:C_0402_1005Metric, symbol Device:C
- added C26, C27, C28, C29: 10n, Capacitor_SMD:C_0402_1005Metric, symbol Device:C
- added D10, D11, D12, D13, D14, D15, D16, D9: 1N5819WS, Diode_SMD:D_SOD-323, symbol Diode:1N5819WS
- added D17, D6, D7, D8: LED, LED_SMD:LED_0603_1608Metric, symbol Device:LED
- added J1: Conn_01x02_Pin, Connector_JST:JST_VH_B2P-VH_1x02_P3.96mm_Vertical, symbol Connector:Conn_01x02_Pin
- added J10, J11, J8, J9: Conn_01x02_Pin, Connector_JST:JST_PH_B2B-PH-K_1x02_P2.00mm_Vertical, symbol Connector:Conn_01x02_Pin
- added J13, J14, J15: Conn_01x03_Pin, Connector_JST:JST_PH_B3B-PH-K_1x03_P2.00mm_Vertical, symbol Connector:Conn_01x03_Pin
- added J17: USB_B_Micro, Connector_USB:USB_Micro-B_Molex-105017-0001, symbol Connector:USB_B_Micro
- added J2: Conn_01x02_Pin, Connector_PinHeader_2.54mm:PinHeader_1x02_P2.54mm_Vertical, symbol Connector:Conn_01x02_Pin
- added R13: 680R, Resistor_SMD:R_0603_1608Metric, symbol Device:R
- added R16, R17, R18, R19, R20, R21, R24: 100, Resistor_SMD:R_0603_1608Metric, symbol Device:R
- added R22: 10k, Resistor_SMD:R_0603_1608Metric, symbol Device:R
- added R26, R27, R28: 330, Resistor_SMD:R_0603_1608Metric, symbol Device:R
- added R31: 1k, Resistor_SMD:R_0603_1608Metric, symbol Device:R
- added TP1, TP10, TP11, TP12, TP13, TP2, TP3, TP4, TP5, TP6, TP7, TP8, TP9: TestPoint, TestPoint:TestPoint_Pad_D1.0mm, symbol Connector:TestPoint
- J12: renamed from J7; footprint (none) -> Connector_JST:JST_PH_B4B-PH-K_1x04_P2.00mm_Vertical
- J16: renamed from J9; footprint (none) -> Connector_JST:JST_PH_B4B-PH-K_1x04_P2.00mm_Vertical
- J18: renamed from J1; value Conn_01x06_Pin -> SWD; footprint (none) -> Connector_JST:JST_PH_B6B-PH-K_1x06_P2.00mm_Vertical
- J3: renamed from J2; footprint (none) -> Connector_JST:JST_PH_B2B-PH-K_1x02_P2.00mm_Vertical
- J4: renamed from J3; footprint (none) -> Connector_JST:JST_PH_B2B-PH-K_1x02_P2.00mm_Vertical
- J5: renamed from J4; footprint (none) -> Connector_JST:JST_PH_B2B-PH-K_1x02_P2.00mm_Vertical
- J6: renamed from J5; footprint (none) -> Connector_JST:JST_VH_B2P-VH_1x02_P3.96mm_Vertical
- J7: renamed from J6; footprint (none) -> Connector_JST:JST_VH_B2P-VH_1x02_P3.96mm_Vertical
- R14, R15: value 5.1k -> 680R
- SW1: footprint easyeda2kicad:SW-SMD_L3.9-W3.0-P4.45 -> ESLThrusterParts:SW-SMD_L3.9-W3.0-P4.45
- U4: renamed from U6; footprint MCP6024-E_SL:SOIC127P600X175-14N -> ESLThrusterParts:SOIC127P600X175-14N
- U5: footprint easyeda2kicad:TSSOP-20_L6.5-W4.4-P0.65-LS6.4-BL -> ESLThrusterParts:TSSOP-20_L6.5-W4.4-P0.65-LS6.4-BL
- U6: renamed from U1; footprint easyeda2kicad:SOIC-8_L4.9-W3.9-P1.27-LS6.0-BL -> ESLThrusterParts:SOIC-8_L4.9-W3.9-P1.27-LS6.0-BL
- renumbered C12 to C1, C5 to C10, C6 to C11, C7 to C12, C8 to C13, C9 to C14, C10 to C15, C11 to C16, C1 to C17, C2 to C18, C3 to C19, C13 to C2, C20 to C21, C21 to C22, C22 to C23, C23 to C25, C16 to C3, C14 to C4, C15 to C5, C17 to C6, C18 to C7, C19 to C8, C4 to C9, D4 to D1, D5 to D2, D1 to D3, D2 to D4, D3 to D5, Q6 to Q1, Q1 to Q2, Q2 to Q3, Q3 to Q4, Q4 to Q5, Q5 to Q6, R2 to R1, R11 to R10, R12 to R11, R18 to R12, R3 to R2, R13 to R23, Rg1 to R25, R16 to R29, R4 to R3, R17 to R30, R5 to R4, R6 to R5, R7 to R6, R8 to R7, R9 to R8, R10 to R9, U4 to U1, U3 to U2, U2 to U3
Connections:
- net VBUS_SENSING is gone; now on net USB_SENSING: R29.2, R30.1
- net +24V: now also TP3.1
- net +3.3V: now also U4.4 (VDD), C20.1, C24.2, D10.1 (K), D12.1 (K), D14.1 (K), D16.1 (K), D6.2 (A), R22.2, TP7.1
- net +5V: now also C30.1, C31.1, C32.1, C33.1, J13.3 (Pin_3), J14.3 (Pin_3), J15.3 (Pin_3), J2.1 (Pin_1), TP5.1; no longer C4.1, C5.1, L1.2, U2.1 (FB)
- net ADC_CLKIN: now also U3.22 (PB10), TP13.1
- net ADC_LOADCELL: now also U3.10 (PA2), U4.1 (VOUTA), U4.2 (VINA-), TP8.1
- net ADC_MISO: now also U3.14 (PA6), TP10.1
- net ADC_MOSI: now also U3.15 (PA7)
- net ADC_SCLK: now also U3.13 (PA5)
- net ADC_~{CS}: now also U3.17 (PB1)
- net ADC_~{DRDY}: now also U3.16 (PB0), TP12.1
- net ADC_~{SYNC}/~{RESET}: now also U3.18 (PB2)
- net GND: now also U4.11 (VSS), U5.9 (AIN3N), C20.2, C24.1, C29.2, C30.2, C31.2, C32.2, C33.2, D11.2 (A), D13.2 (A), D15.2 (A), D9.2 (A), J1.2 (Pin_2), J11.2 (Pin_2), J13.1 (Pin_1), J14.1 (Pin_1), J15.1 (Pin_1), J17.5 (GND), J17.6 (Shield), R13.2, R31.2, TP11.1, TP9.1
- net GPIO1_Valve: now also U3.40 (PB3)
- net GPIO2_Valve: now also U3.41 (PB4)
- net GPIO3_Valve: now also U3.42 (PB5)
- net GPIO4_Heater: now also U3.43 (PB6)
- net GPIO5_Heater: now also U3.44 (PB7)
- net UART_RX: now also U3.32 (PA10)
- net UART_TX: now also U3.31 (PA9)
- net USB_DP: now also J17.3 (D+)
- net VBUS: now also J1.1 (Pin_1), TP1.1
- net S_OUT2: now reaches U4.10 (VINC+)
- net S_OUT2: now also D13.1 (K), D14.2 (A), R27.1
- net S_OUT3: now reaches U4.12 (VIND+)
- net S_OUT3: now also D15.1 (K), D16.2 (A), R28.1
- net ADC_PRESSURE3: now reaches U4.13 (VIND-)
- net ADC_PRESSURE3: now also U3.11 (PA3), U4.14 (VOUTD), TP2.1
- net at U4.3 (VINA+): now also D10.2 (A), D9.1 (K), R24.2
- net S_OUT1: now reaches U4.5 (VINB+)
- net S_OUT1: now also D11.1 (K), D12.2 (A), R26.1
- net ADC_PRESSURE1: now reaches U4.6 (VINB-)
- net ADC_PRESSURE1: now also U3.9 (PA1), U4.7 (VOUTB), TP6.1
- net ADC_PRESSURE2: now reaches U4.8 (VOUTC)
- net ADC_PRESSURE2: now also U3.12 (PA4), U4.9 (VINC-), TP4.1
- net at U5.10 (AIN3P): now also C29.1, J11.1 (Pin_1), R22.1
- net at U5.3 (AIN0P): now also C26.1, R16.2
- net at U5.4 (AIN0N): now also C26.2, R17.2
- net at U5.5 (AIN1N): now also C27.1, R18.2
- net at U5.6 (AIN1P): now also C27.2, R19.2
- net at U5.7 (AIN2P): now also C28.1, R20.2
- net at U5.8 (AIN2N): now also C28.2, R21.2
- net at R29.1: now also D17.2 (A), J17.1 (VBUS)
- net at U6.6 (VO): now also R24.1
- net at R14.1: now also D7.1 (K)
- net at R15.1: now also D8.1 (K)
- net DEBUG_1: now reaches U3.25 (PB11)
- net DEBUG_1: now also D7.2 (A)
- net DEBUG_2: now reaches U3.26 (PB12)
- net DEBUG_2: now also D8.2 (A)
- net USB_SENSING: now reaches U3.30 (PA8)
- net SWO: no longer names the net of J18.6 (Pin_6)
- net SWO: no longer U3.40 (PB3)
- net USB_DM renamed USB_DN
- net USB_DN: now also J17.2 (D-)
- new net: J13.2 (Pin_2), R26.2
- new net: J8.2 (Pin_2), R17.1
- new net: D6.1 (K), R13.1
- new net: C4.1, C5.1, J2.2 (Pin_2), L1.2, U2.1 (FB)
- new net: J10.2 (Pin_2), R21.1
- new net: J8.1 (Pin_1), R16.1
- new net: J10.1 (Pin_1), R20.1
- new net: J9.1 (Pin_1), R19.1
- new net: D17.1 (K), R31.1
- new net: J14.2 (Pin_2), R27.2
- new net: J9.2 (Pin_2), R18.1
- new net: J15.2 (Pin_2), R28.2
- no-connect marks 10 -> 11
Other:
- note added: "BLACK"
- note added: "CL=2*(CLO-Cs)=2*(20-5)=30pF"
- note added: "Comms"
- note added: "Debug LEDs"
- note added: "G = 5 + (80000/R)"
- note added: "GREEN"
- note added: "RED"
- note added: "Test Pads"
- note added: "WHITE"
- note removed: "BLACK_EXCITATION-"
- note removed: "CL=2*(CLO-Cs) =2*(20 - 5) =30pF"
- note removed: "G = 5 + (80000/Rg)"
- note removed: "GREEN_SIGNAL+"
- note removed: "RED_EXCITATION+"
- note removed: "Serial Wire Debug Interface"
- note removed: "WHITE_SIGNAL-"
- company: (none) -> Stellenbosch University
- title: (none) -> Thruster V3 PCB
- moved on the sheet: C10, C11, C12, C13, C14, C15, C16, C17, C18, C19, C21, C22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
